File: kicad/carpc.sch (KiCad schematic (older format))
At the start: 64 parts, among them IC1 MEGA8-P, IC2 MAX232, IC2 VCC, K1 K1, K2 K2, K3 K3, K6 K6, T1 2SC458, T2 2SC458, T4 2SC458

Commit message: fixed conversion errors (relays)
Parts:
- removed IC2: VCC, IC2P, symbol IC_MAX232
- removed K1, K2, K3, K6: (no value), symbol K_JS-M1*
- removed K1: K1, symbol K_JS-M1*
- removed K2: K2, symbol K_JS-M1*
- removed K3: K3, symbol K_JS-M1*
- removed K6: K6, symbol K_JS-M1*
- removed SUPPLY1, SUPPLY10, SUPPLY11, SUPPLY12, SUPPLY13, SUPPLY14, SUPPLY15, SUPPLY16, SUPPLY17, SUPPLY2, SUPPLY3, SUPPLY4, SUPPLY5, SUPPLY6, SUPPLY7, SUPPLY8, SUPPLY9: (no value), symbol SUPPLY_GND
- added GND (x17): (no value), symbol SUPPLY_GND
- added K1, K2, K3, K6: RELAY-1XCHANCE, symbol RELAY-1XCHANCE
Connections:
- net labels added: 12V, K1 Change, K1 Close if active, K2 C, K2 NO
- wire segments 168 -> 157

Commit message: changed connectors for 12V input and ext. Battery
Parts:
- removed 1, 2: 130k, symbol R_R-EU_
- removed 12V: (no value), symbol P+_VCC
- removed C: 3.3uF, symbol C_C
- removed D1: 1N5400, symbol D_1N5400
- removed D5: BZW04XX, symbol D_BZW04XX
- removed GND (x17): (no value), symbol SUPPLY_GND
- removed IC1: MEGA8-P, symbol IC_MEGA8-P
- removed IC2: MAX232, symbol IC_MAX232
- removed L4940-5V: 2N5496, symbol T_2N5496
- removed R: 10k, symbol R_R-EU_
- removed SV1: (no value), symbol SV_MA05-2
- removed SV5: (no value), symbol SV_MA10-1
- removed T4: 2SC458, symbol T_2SC458
- added 11, 21: 130k, symbol R_R-EU_
- added 12V1: ~, symbol P+_VCC
- added C6: 10u, symbol C_C
- added D1: BZW04XX, symbol D_BZW04XX
- added D5: 1N5400, symbol D_1N5400
- added GND1, GND10, GND11, GND12, GND13, GND14, GND15, GND16, GND17, GND2, GND3, GND4, GND5, GND6, GND8, GND9: ~, symbol SUPPLY_GND
- added IC1: MAX232, symbol IC_MAX232
- added IC2: MEGA8-P, symbol IC_MEGA8-P
- added L4940-5V1: 2N5496, symbol T_2N5496
- added P1, P2, P?: CONN_2, symbol CONN_2
- added R9: 470, symbol R_R-EU_
- added SV2: ~, symbol SV_MA05-2
- added T3: 2SC458, symbol T_2SC458
- C1: value 10u -> 100n
- C2: value 100n -> 10u
- C4: value 10u -> 3.3uF
- LED1, LED2, S1, S2, SV3, SV4, X1: value (none) -> ~
- R1: value 10k -> 100
- R2, R3: value 470 -> 10k
- R4: value 130k -> 10k
- R5: value 470 -> 180k
- R6: value 10k -> 130k
- R7: value 100 -> 470
- R8: value 180k -> 470
- renumbered K2 to K1, K3 to K2, K1 to K3, K6 to K4
Connections:
- wire segments 157 -> 147
Other:
- moved on the sheet: K1

Commit message: changed connectors for other relays
Parts:
- removed SV4: ~, symbol SV_MA20-1
- added P? (x3): CONN_2, symbol CONN_2
Connections:
- wire segments 147 -> 136

Commit message: added crystal & annotation
Parts:
- added X?: CRYSTAL, symbol CRYSTAL
Connections:
- wire segments 136 -> 138
