File: kicad/carpc.sch (KiCad schematic (older format))
At the start: 63 parts, among them IC1 MAX232, IC2 MEGA8-P, K1 RELAY-1XCHANCE, K2 RELAY-1XCHANCE, K3 RELAY-1XCHANCE, K4 RELAY-1XCHANCE, P1 CONN_2, P2 CONN_2, T1 2SC458, T2 2SC458, T3 2SC458

Commit message: fixed 12V issue
Parts:
- removed 12V1: ~, symbol P+_VCC
Connections:
- net labels removed: VCC
Changed lines of the file:
@@
-EESchema Schematic File Version 2  date Wed 03 Oct 2012 11:02:27 PM CEST
+EESchema Schematic File Version 2  date Wed 03 Oct 2012 11:55:49 PM CEST
 LIBS:74xx
 LIBS:adc-dac
@@
 Comment4 ""
 $EndDescr
+Text Label 3300 3000 2    60   ~ 0
+12V
 Wire Wire Line
 	3750 6550 3900 6550
@@
 	-1   0    0    1
 $EndComp
-Text Label 4200 4200 0    60   ~ 0
+Text Label 4200 4200 2    60   ~ 0
 K2 NO
 Text Label 4200 5050 0    60   ~ 0
@@
 	1    7400 7250
 	-1   0    0    1
-$EndComp
-$Comp
-L P+_VCC 12V1
-U 1 1 506BAD2B
-P 3200 3000
-F 0 "12V1" V 3100 2900 70  0000 L BNN
-F 1 "~" H 3200 3000 60  0001 C CNN
-	1    3200 3000
-	0    -1   -1   0
 $EndComp
 $Comp
@@
 Text Label 6600 6250 0    70   ~ 0
 TXD
-Text Label 4200 3000 0    70   ~ 0
-VCC
-Text Label 1250 3200 0    70   ~ 0
-12V
 Text Label 2800 5550 0    70   ~ 0
 12V

Commit message: Removed MAX232, TTL to Pins on SV3
Parts:
- removed C3, C5, C6: 10u, symbol C_C
- removed GND8: ~, symbol SUPPLY_GND
- removed IC1: MAX232, symbol IC_MAX232
- removed X1: ~, symbol X_F09
- removed X?: CRYSTAL, symbol CRYSTAL
Connections:
- wire segments 138 -> 124

Commit message: Rearranged
Parts:
- removed C2: 10u, symbol C_C
Connections:
- wire segments 124 -> 122
Other:
- moved on the sheet: K1, P1, P2, P?

Commit message: added netlist (kicad)
Parts:
- gave numbers to parts that had none: 4
- renumbered 11 to 1, 21 to 2, C4 to C2, GND3 to GND1, GND13 to GND10, GND14 to GND11, GND10 to GND12, GND15 to GND13, GND16 to GND14, GND17 to GND15, GND1 to GND2, GND4 to GND3, GND5 to GND4, GND6 to GND5, GND2 to GND6, GND9 to GND7, GND11 to GND8, GND12 to GND9, IC2 to IC1, SV2 to ISP_SOCKET1, L4940-5V1 to L1, SV3 to PinSocket1, R2 to R1, R3 to R2, R1 to R3
Changed lines of the file:
@@
-EESchema Schematic File Version 2  date Thu 04 Oct 2012 12:38:22 AM CEST
+EESchema Schematic File Version 2  date Thu 04 Oct 2012 01:05:06 AM CEST
 LIBS:74xx
 LIBS:adc-dac
@@
 12V
 $Comp
-L CONN_2 P?
+L CONN_2 P6
 U 1 1 506BB096
 P 10950 4700
-F 0 "P?" V 10900 4700 40  0000 C CNN
+F 0 "P6" V 10900 4700 40  0000 C CNN
 F 1 "CONN_2" V 11000 4700 40  0000 C CNN
 	1    10950 4700
@@
 $EndComp
 $Comp
-L CONN_2 P?
+L CONN_2 P4
 U 1 1 506BB075
 P 10400 900
-F 0 "P?" V 10350 900 40  0000 C CNN
+F 0 "P4" V 10350 900 40  0000 C CNN
 F 1 "CONN_2" V 10450 900 40  0000 C CNN
 	1    10400 900
@@
 $EndComp
 $Comp
-L CONN_2 P?
+L CONN_2 P5
 U 1 1 506BB029
 P 10700 2950
-F 0 "P?" V 10650 2950 40  0000 C CNN
+F 0 "P5" V 10650 2950 40  0000 C CNN
 F 1 "CONN_2" V 10750 2950 40  0000 C CNN
 	1    10700 2950
@@
 GND
 $Comp
-L CONN_2 P?
+L CONN_2 P3
 U 1 1 506BAFC8
 P 1100 2000
-F 0 "P?" V 1050 2000 40  0000 C CNN
+F 0 "P3" V 1050 2000 40  0000 C CNN
 F 1 "CONN_2" V 1150 2000 40  0000 C CNN
 	1    1100 2000
@@
 $EndComp
 $Comp
-L R_R-EU_ 11
+L R_R-EU_ 1
 U 1 1 506BAD29
 P 5300 6850
-F 0 "11" H 5150 6908 70  0000 L BNN
+F 0 "1" H 5150 6908 70  0000 L BNN
 F 1 "130k" H 5150 6720 70  0000 L BNN
 	1    5300 6850
@@
 $EndComp
 $Comp
-L R_R-EU_ 21
+L R_R-EU_ 2
 U 1 1 506BAD2A
 P 5300 7050
-F 0 "21" H 5150 7108 70  0000 L BNN
+F 0 "2" H 5150 7108 70  0000 L BNN
 F 1 "130k" H 5150 6920 70  0000 L BNN
 	1    5300 7050
@@
 $EndComp
 $Comp
-L C_C C4
+L C_C C2
 U 1 1 506BAD2C
 P 2100 6550
-F 0 "C4" H 2160 6564 70  0000 L BNN
+F 0 "C2" H 2160 6564 70  0000 L BNN
 F 1 "3.3uF" H 2159 6365 70  0000 L BNN
 	1    2100 6550
@@
 $EndComp
 $Comp
-L IC_MEGA8-P IC2
+L IC_MEGA8-P IC1
 U 1 1 506BAD36
 P 3200 6150
-F 0 "IC2" H 2500 4750 70  0000 L BNN
+F 0 "IC1" H 2500 4750 70  0000 L BNN
 F 1 "MEGA8-P" H 2501 7400 70  0000 L BNN
 	1    3200 6150
@@
 $EndComp
 $Comp
-L T_2N5496 L4940-5V1
+L T_2N5496 L1
 U 1 1 506BAD38
 P 6850 1250
-F 0 "L4940-5V1" H 6450 1550 70  0000 L BNN
+F 0 "L1" H 6450 1550 70  0000 L BNN
 F 1 "2N5496" H 6450 1450 70  0000 L BNN
 	1    6850 1250
@@
 $EndComp
 $Comp
-L R_R-EU_ R2
+L R_R-EU_ R1
 U 1 1 506BAD3B
 P 1100 5350
-F 0 "R2" H 950 5409 70  0000 L BNN
+F 0 "R1" H 950 5409 70  0000 L BNN
 F 1 "10k" H 950 5220 70  0000 L BNN
 	1    1100 5350
@@
 $EndComp
 $Comp
-L R_R-EU_ R3
+L R_R-EU_ R2
 U 1 1 506BAD3C
 P 1800 5050
-F 0 "R3" H 1650 5109 70  0000 L BNN
+F 0 "R2" H 1650 5109 70  0000 L BNN
 F 1 "10k" H 1650 4920 70  0000 L BNN
 	1    1800 5050
@@
 $EndComp
 $Comp
-L R_R-EU_ R1
+L R_R-EU_ R3
 U 1 1 506BAD0B
 P 2950 2100
-F 0 "R1" H 2800 2159 70  0000 L BNN
+F 0 "R3" H 2800 2159 70  0000 L BNN
 F 1 "100" H 2800 1970 70  0000 L BNN
 	1    2950 2100
@@
 $EndComp
 $Comp
-L SUPPLY_GND GND4
+L SUPPLY_GND GND3
 U 1 1 506BAD10
 P 2000 5250
-F 0 "GND4" H 1926 5125 70  0000 L BNN
+F 0 "GND3" H 1926 5125 70  0000 L BNN
 F 1 "~" H 2000 5250 60  0001 C CNN
 	1    2000 5250
@@
 $EndComp
 $Comp
-L SUPPLY_GND GND5
+L SUPPLY_GND GND4
 U 1 1 506BAD11
 P 2000 6250
-F 0 "GND5" H 1926 6125 70  0000 L BNN
+F 0 "GND4" H 1926 6125 70  0000 L BNN
 F 1 "~" H 2000 6250 60  0001 C CNN
 	1    2000 6250
@@
 $EndComp
 $Comp
-L SUPPLY_GND GND3
+L SUPPLY_GND GND1
 U 1 1 506BAD12
 P 1400 5850
-F 0 "GND3" H 1325 5725 70  0000 L BNN
+F 0 "GND1" H 1325 5725 70  0000 L BNN
 F 1 "~" H 1400 5850 60  0001 C CNN
 	1    1400 5850
@@
 $EndComp
 $Comp
-L SUPPLY_GND GND6
+L SUPPLY_GND GND5
 U 1 1 506BAD13
 P 2100 6850
-F 0 "GND6" H 2025 6725 70  0000 L BNN
+F 0 "GND5" H 2025 6725 70  0000 L BNN
 F 1 "~" H 2100 6850 60  0001 C CNN
 	1    2100 6850
@@
 $EndComp
 $Comp
-L SUPPLY_GND GND10
+L SUPPLY_GND GND12
 U 1 1 506BAD14
 P 8450 1900
-F 0 "GND10" H 8375 1775 70  0000 L BNN
+F 0 "GND12" H 8375 1775 70  0000 L BNN
 F 1 "~" H 8450 1900 60  0001 C CNN
 	1    8450 1900
@@
 $EndComp
 $Comp
-L SUPPLY_GND GND1
+L SUPPLY_GND GND2
 U 1 1 506BAD15
 P 1450 1200
-F 0 "GND1" H 1375 1075 70  0000 L BNN
+F 0 "GND2" H 1375 1075 70  0000 L BNN
 F 1 "~" H 1450 1200 60  0001 C CNN
 	1    1450 1200
@@
 $EndComp
 $Comp
-L SUPPLY_GND GND16
+L SUPPLY_GND GND14
 U 1 1 506BAD16
 P 9500 5050
-F 0 "GND16" H 9425 4925 70  0000 L BNN
+F 0 "GND14" H 9425 4925 70  0000 L BNN
 F 1 "~" H 9500 5050 60  0001 C CNN
 	1    9500 5050
@@
 $EndComp
 $Comp
-L SUPPLY_GND GND17
+L SUPPLY_GND GND15
 U 1 1 506BAD17
 P 9500 7050
-F 0 "GND17" H 9425 6925 70  0000 L BNN
+F 0 "GND15" H 9425 6925 70  0000 L BNN
 F 1 "~" H 9500 7050 60  0001 C CNN
 	1    9500 7050
@@
 $EndComp
 $Comp
-L SUPPLY_GND GND2
+L SUPPLY_GND GND6
 U 1 1 506BAD18
 P 3250 3000
-F 0 "GND2" H 3175 2875 70  0000 L BNN
+F 0 "GND6" H 3175 2875 70  0000 L BNN
 F 1 "~" H 3250 3000 60  0001 C CNN
 	1    3250 3000
@@
 $EndComp
 $Comp
-L SUPPLY_GND GND15
+L SUPPLY_GND GND13
 U 1 1 506BAD0A
 P 9500 3050
-F 0 "GND15" H 9425 2925 70  0000 L BNN
+F 0 "GND13" H 9425 2925 70  0000 L BNN
 F 1 "~" H 9500 3050 60  0001 C CNN
 	1    9500 3050
@@
 $EndComp
 $Comp
-L SUPPLY_GND GND14
+L SUPPLY_GND GND11
 U 1 1 506BAD1A
 P 5700 6050
-F 0 "GND14" H 5625 5925 70  0000 L BNN
+F 0 "GND11" H 5625 5925 70  0000 L BNN
 F 1 "~" H 5700 6050 60  0001 C CNN
 	1    5700 6050
@@
 $EndComp
 $Comp
-L SUPPLY_GND GND9
+L SUPPLY_GND GND7
 U 1 1 506BAD1C
 P 5000 5650
-F 0 "GND9" H 4926 5525 70  0000 L BNN
+F 0 "GND7" H 4926 5525 70  0000 L BNN
 F 1 "~" H 5000 5650 60  0001 C CNN
 	1    5000 5650
@@
 $EndComp
 $Comp
-L SUPPLY_GND GND11
+L SUPPLY_GND GND8
 U 1 1 506BAD1D
 P 5400 5650
-F 0 "GND11" H 5326 5525 70  0000 L BNN
+F 0 "GND8" H 5326 5525 70  0000 L BNN
 F 1 "~" H 5400 5650 60  0001 C CNN
 	1    5400 5650
@@
 $EndComp
 $Comp
-L SUPPLY_GND GND13
+L SUPPLY_GND GND10
 U 1 1 506BAD1E
 P 5600 7050
-F 0 "GND13" H 5525 6925 70  0000 L BNN
+F 0 "GND10" H 5525 6925 70  0000 L BNN
 F 1 "~" H 5600 7050 60  0001 C CNN
 	1    5600 7050
@@
 $EndComp
 $Comp
-L SUPPLY_GND GND12
+L SUPPLY_GND GND9
 U 1 1 506BAD1F
 P 5600 6850
-F 0 "GND12" H 5525 6725 70  0000 L BNN
+F 0 "GND9" H 5525 6725 70  0000 L BNN
 F 1 "~" H 5600 6850 60  0001 C CNN
 	1    5600 6850
@@
 $EndComp
 $Comp
-L SV_MA05-2 SV2
+L SV_MA05-2 ISP_SOCKET1
 U 1 1 506BAD20
 P 8050 1300
-F 0 "SV2" H 7900 1630 70  0000 L BNN
+F 0 "ISP_SOCKET1" H 7900 1630 70  0000 L BNN
 F 1 "~" H 8050 1300 60  0001 C CNN
 	1    8050 1300
@@
 $EndComp
 $Comp
-L SV_MA08-2 SV3
+L SV_MA08-2 PinSocket1
 U 1 1 506BAD21
 P 5000 3850
-F 0 "SV3" H 4851 4380 70  0000 L BNN
+F 0 "PinSocket1" H 4851 4380 70  0000 L BNN
 F 1 "~" H 5000 3850 60  0001 C CNN
 	1    5000 3850

Commit message: fixed annotation
Parts:
- renumbered R8 to R10, R9 to R11, 1 to R5, 2 to R6, R5 to R7, R6 to R8, R7 to R9
Changed lines of the file:
@@
-EESchema Schematic File Version 2  date Thu 04 Oct 2012 01:05:06 AM CEST
+EESchema Schematic File Version 2  date Thu 04 Oct 2012 01:08:25 AM CEST
 LIBS:74xx
 LIBS:adc-dac
@@
 $EndComp
 $Comp
-L R_R-EU_ 1
+L R_R-EU_ R5
 U 1 1 506BAD29
 P 5300 6850
-F 0 "1" H 5150 6908 70  0000 L BNN
+F 0 "R5" H 5150 6908 70  0000 L BNN
 F 1 "130k" H 5150 6720 70  0000 L BNN
 	1    5300 6850
@@
 $EndComp
 $Comp
-L R_R-EU_ 2
+L R_R-EU_ R6
 U 1 1 506BAD2A
 P 5300 7050
-F 0 "2" H 5150 7108 70  0000 L BNN
+F 0 "R6" H 5150 7108 70  0000 L BNN
 F 1 "130k" H 5150 6920 70  0000 L BNN
 	1    5300 7050
@@
 $EndComp
 $Comp
-L R_R-EU_ R8
+L R_R-EU_ R10
 U 1 1 506BAD3D
 P 9100 4650
-F 0 "R8" H 8950 4709 70  0000 L BNN
+F 0 "R10" H 8950 4709 70  0000 L BNN
 F 1 "470" H 8950 4520 70  0000 L BNN
 	1    9100 4650
@@
 $EndComp
 $Comp
-L R_R-EU_ R9
+L R_R-EU_ R11
 U 1 1 506BAD3E
 P 9100 6650
-F 0 "R9" H 8950 6709 70  0000 L BNN
+F 0 "R11" H 8950 6709 70  0000 L BNN
 F 1 "470" H 8950 6520 70  0000 L BNN
 	1    9100 6650
@@
 $EndComp
 $Comp
-L R_R-EU_ R6
+L R_R-EU_ R8
 U 1 1 506BAD3F
 P 5700 5750
-F 0 "R6" H 5550 5809 70  0000 L BNN
+F 0 "R8" H 5550 5809 70  0000 L BNN
 F 1 "130k" H 5550 5620 70  0000 L BNN
 	1    5700 5750
@@
 $EndComp
 $Comp
-L R_R-EU_ R7
+L R_R-EU_ R9
 U 1 1 506B9CCB
 P 9100 2650
-F 0 "R7" H 8950 2709 70  0000 L BNN
+F 0 "R9" H 8950 2709 70  0000 L BNN
 F 1 "470" H 8950 2520 70  0000 L BNN
 	1    9100 2650
@@
 $EndComp
 $Comp
-L R_R-EU_ R5
+L R_R-EU_ R7
 U 1 1 506BAD0C
 P 5700 5250
-F 0 "R5" H 5550 5309 70  0000 L BNN
+F 0 "R7" H 5550 5309 70  0000 L BNN
 F 1 "180k" H 5550 5120 70  0000 L BNN
 	1    5700 5250
