File: kicad/carpc.sch (KiCad schematic (older format))
At the start: 54 parts, among them IC1 MEGA8-P, K1 RELAY-1XCHANCE, K2 RELAY-1XCHANCE, K3 RELAY-1XCHANCE, K4 RELAY-1XCHANCE, P1 CONN_2, P2 CONN_2, P3 CONN_2, P4 CONN_2, P5 CONN_2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

Commit message: Finialising some stuff
Parts:
- removed GND11, GND7, GND8: ~, symbol SUPPLY_GND
Connections:
- wire segments 122 -> 128
Other:
- note added: "12V from Car"
Changed lines of the file:
@@
-EESchema Schematic File Version 2  date Fri 05 Oct 2012 09:30:10 PM CEST
+EESchema Schematic File Version 2  date Sun 14 Oct 2012 08:23:47 AM CEST
 LIBS:74xx
 LIBS:adc-dac
@@
 Sheet 1 1
 Title "carpc.sch"
-Date "5 oct 2012"
+Date "14 oct 2012"
 Rev "1.0"
 Comp ""
@@
 Comment4 ""
 $EndDescr
+Connection ~ 5400 5750
+Wire Wire Line
+	5700 5950 5500 5950
+Wire Wire Line
+	5500 5750 5500 5950
+Wire Wire Line
+	5000 5750 5500 5750
+Connection ~ 5000 6150
+Wire Wire Line
+	5100 6150 4200 6150
+Connection ~ 5100 5750
+Wire Wire Line
+	5100 5750 5100 5650
 Wire Wire Line
 	8700 6350 8700 4650
@@
 	5300 6250 5300 6150
 Wire Wire Line
-	4200 6150 5000 6150
-Wire Wire Line
 	4700 3850 4400 3850
 Wire Wire Line
@@
 Wire Wire Line
 	8900 6650 4200 6650
+Wire Wire Line
+	5100 5650 4850 5650
+Connection ~ 5300 5750
+Wire Wire Line
+	5300 6150 5400 6150
+Text Label 4850 5650 2    60   ~ 0
+GND
+Text Notes 1600 850  0    60   ~ 0
+12V from Car
 Text Label 5500 3750 0    60   ~ 0
 TXD
@@
 $EndComp
 $Comp
-L SUPPLY_GND GND11
-U 1 1 506BAD1A
-P 5700 6050
-F 0 "GND11" H 5625 5925 70  0000 L BNN
-F 1 "~" H 5700 6050 60  0001 C CNN
-	1    5700 6050
-	1    0    0    -1
-$EndComp
-$Comp
-L SUPPLY_GND GND7
-U 1 1 506BAD1C
-P 5000 5650
-F 0 "GND7" H 4926 5525 70  0000 L BNN
-F 1 "~" H 5000 5650 60  0001 C CNN
-	1    5000 5650
-	-1   0    0    1
-$EndComp
-$Comp
-L SUPPLY_GND GND8
-U 1 1 506BAD1D
-P 5400 5650
-F 0 "GND8" H 5326 5525 70  0000 L BNN
-F 1 "~" H 5400 5650 60  0001 C CNN
-	1    5400 5650
-	-1   0    0    1
-$EndComp
-$Comp
